File: cell_sim_relay_board/cell_sim_relay_board.kicad_pcb (KiCad board)
At the start: 2 copper layers, 100 x 100 mm, 76 parts, among them J1 1843787, J2 JST_03, J3 JST_03, J4 Barrel_Jack_Switch, J5 1843787, K1 FINDER-34.51, K10 FINDER-34.51, K11 FINDER-34.51, K12 FINDER-34.51, K13 FINDER-34.51, K14 FINDER-34.51, K15 FINDER-34.51, K16 FINDER-34.51, K17 FINDER-34.51, K18 FINDER-34.51, K19 FINDER-34.51, K2 FINDER-34.51, K20 FINDER-34.51, K21 FINDER-34.51, K22 FINDER-34.51, K23 FINDER-34.51, K24 FINDER-34.51, K25 FINDER-34.51, K26 FINDER-34.51, K27 FINDER-34.51, K28 FINDER-34.51, K3 FINDER-34.51, K4 FINDER-34.51, K5 FINDER-34.51, K6 FINDER-34.51, K7 FINDER-34.51, K8 FINDER-34.51, K9 FINDER-34.51, U1 ULN2003, U2 ULN2003, U3 ULN2003, U4 ULN2003, U5 MCP23017_SO, U6 MCP23017_SO, U7 LM1117MP-3.3

Commit message: update
Parts:
- added REF**: KiCad-Logo2_6mm_SilkScreen, Symbol:KiCad-Logo2_6mm_SilkScreen, F.Cu at (159.0, 120.0)
- added REF**: OSHW-Logo2_9.8x8mm_SilkScreen, Symbol:OSHW-Logo2_9.8x8mm_SilkScreen, F.Cu at (173.5, 121.0)
- moved C4 14.9 mm to (147.0, 46.6), turned to 180 degrees
- moved C9 2.86 mm to (137.7, 115.5)
Routing:
- net PWR_12V: track 713.9 -> 700.6 mm
- net PWR_GND: track 331.7 -> 320.3 mm
- net PWR_5V: track 140.0 -> 137.5 mm, vias 10 -> 20
- net /Relay_channel1/cntrl_cell_open: track 15.5 -> 17.1 mm
- net /Relay_channel/cntrl_cell_open: track 18.6 -> 20.1 mm
- net /Relay_channel/cntrl_cell_short: track 47.0 -> 48.2 mm
- net /Relay_channel12/cntrl_cell_open: track 14.8 -> 15.8 mm
- net /Relay_channel1/cntrl_cell_short: track 45.6 -> 46.6 mm
- net /Relay_channel11/cntrl_cell_open: track 16.6 -> 15.8 mm
- net /OUT_CELL_12(short)+: track 35.3 -> 34.6 mm
- net /Relay_channel11/cntrl_cell_short: track 45.9 -> 46.6 mm
Other:
- board text added: "5V"
- board text added: "Cell voltage monitoring Falul injection device V1 - 13 chennals"
- board text added: "FINDER-34.51"
- board text added: "INPUT"
- board text added: "OUT"
- board text added: "Sofia, Bulgaria, 2026"
- board text added: "address"
- board text added: "https://github.com/ami3go"
