File: 12x_relay_board/12x_relay_board.kicad_pcb (KiCad board)
At the start: 2 copper layers, 100 x 100 mm, 46 parts, among them J1 Conn_01x36_MountingPin, J2 JST_03, J3 JST_03, J4 Barrel_Jack_Switch, K1 FINDER-34.51, K10 FINDER-34.51, K11 FINDER-34.51, K12 FINDER-34.51, K2 FINDER-34.51, K3 FINDER-34.51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

Commit message: update
Parts:
- added J5: Conn_01x09, TerminalBlock:TerminalBlock_Xinya_XY308-2.54-9P_1x09_P2.54mm_Horizontal, F.Cu at (212.6, 57.2)
- added J6: Conn_01x09, TerminalBlock:TerminalBlock_Xinya_XY308-2.54-9P_1x09_P2.54mm_Horizontal, F.Cu at (212.6, 75.2)
- added J7: Conn_01x09, TerminalBlock:TerminalBlock_Xinya_XY308-2.54-9P_1x09_P2.54mm_Horizontal, F.Cu at (212.6, 93.2)
- added J8: Conn_01x09, TerminalBlock:TerminalBlock_Xinya_XY308-2.54-9P_1x09_P2.54mm_Horizontal, F.Cu at (212.6, 111.2)
- added K13: FINDER-34.51, Relay_THT:Relay_SPDT_Finder_34.51_Vertical, F.Cu at (163.9, 111.0)
- added K14: FINDER-34.51, Relay_THT:Relay_SPDT_Finder_34.51_Vertical, F.Cu at (163.9, 117.8)
- J1: value Conn_01x36_MountingPin -> Conn_01x09; footprint Connector_PinHeader_2.54mm:PinHeader_1x36_P2.54mm_Vertical -> TerminalBlock:TerminalBlock_Xinya_XY308-2.54-9P_1x09_P2.54mm_Horizontal
- moved J1 14.8 mm to (212.6, 39.2), turned to 180 degrees
- moved K12 14.6 mm to (163.9, 104.2)
- moved K11 13.5 mm to (163.9, 97.4)
- moved K10 12.3 mm to (163.9, 90.6)
- moved K9 11.2 mm to (163.9, 83.8)
- moved U5 10.6 mm to (137.4, 75.0)
- moved K8 10.2 mm to (163.9, 77.0)
- moved K7 9.14 mm to (163.9, 70.2)
- moved K6 8.15 mm to (163.9, 63.4)
- moved K5 7.22 mm to (163.9, 56.6)
- moved K4 6.38 mm to (163.9, 49.8)
- moved K3 5.68 mm to (163.9, 43.0)
- moved K2 5.16 mm to (163.9, 36.2)
- moved K1 4.89 mm to (163.9, 29.4)
Connections:
- J1 pad 1: /Relay_channel_1/NC -> /Relay_channel_1/NO
- J1 pad 3: /Relay_channel_1/NO -> /Relay_channel_1/NC
- J1 pad 4: /Relay_channel_2/NC -> /Relay_channel_2/NO
- J1 pad 6: /Relay_channel_2/NO -> /Relay_channel_2/NC
- J1 pad 7: /Relay_channel_3/NC -> /Relay_channel_3/NO
- J1 pad 9: /Relay_channel_3/NO -> /Relay_channel_3/NC
- U2 pad 10: /Relay_driver1/OUT7 -> /Relay_channel_14/cntrl_A1
- U2 pad 11: /Relay_driver1/OUT6 -> /Relay_channel_13/cntrl_A1
Routing:
- net PWR_12V: track 55.1 -> 140.2 mm
- net /Relay_channel_4/COM: track 0.00 -> 39.0 mm
- net /Relay_channel_1/NC: track 0.00 -> 38.4 mm
- net /Relay_channel_4/NC: track 0.00 -> 37.4 mm
- net /Relay_channel_1/COM: track 0.00 -> 35.6 mm
- net /Relay_channel_4/NO: track 0.00 -> 33.6 mm
- net /Relay_channel_1/NO: track 0.00 -> 33.0 mm
- net /Relay_channel_11/NC: track 0.00 -> 31.3 mm
- net PWR_GND: track 152.8 -> 121.5 mm
- net /Relay_channel_7/cntrl_A1: track 36.7 -> 6.88 mm
- net /Relay_channel_2/NC: track 0.00 -> 29.1 mm
- net /Relay_channel_2/COM: track 0.00 -> 26.6 mm
- net /Relay_channel_5/NC: track 0.00 -> 25.5 mm
- net (no net): track 15.9 -> 41.2 mm
- net /Relay_channel_2/NO: track 0.00 -> 24.5 mm
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
Commit message: update
Parts:
- added C1: 100nF, PCM_JLCPCB:C_0603, F.Cu at (151.0, 89.3)
- added C13: 1uF, PCM_JLCPCB:C_0603, F.Cu at (119.0, 75.5)
- added C14: 100nF, PCM_JLCPCB:C_0603, F.Cu at (119.0, 74.1)
- added C15: 100nF, PCM_JLCPCB:C_0603, F.Cu at (119.0, 72.7)
- added C16: 1uF, PCM_JLCPCB:C_0603, F.Cu at (119.0, 71.2)
- added C5: 100nF, PCM_JLCPCB:C_0603, F.Cu at (151.0, 91.6)
- added C6: 100nF, PCM_JLCPCB:C_0603, F.Cu at (151.0, 93.8)
- added D4: BAV23C, Package_TO_SOT_SMD_AKL:SOT-23, F.Cu at (136.0, 58.1)
- added J9: Conn_01x08, Connector_PinHeader_2.54mm:PinHeader_2x04_P2.54mm_Vertical, F.Cu at (144.2, 90.5)
- added K15: FINDER-34.51, Relay_THT:Relay_SPDT_Finder_34.51_Vertical, F.Cu at (163.9, 116.2)
- added LED1: LED_0603, LED_SMD_AKL:LED_0603_1608Metric, F.Cu at (157.0, 29.3)
- added LED10: LED_0603, LED_SMD_AKL:LED_0603_1608Metric, F.Cu at (157.0, 85.1)
- added LED11: LED_0603, LED_SMD_AKL:LED_0603_1608Metric, F.Cu at (157.0, 91.3)
- added LED12: LED_0603, LED_SMD_AKL:LED_0603_1608Metric, F.Cu at (157.0, 97.5)
- added LED13: LED_0603, LED_SMD_AKL:LED_0603_1608Metric, F.Cu at (157.0, 103.7)
- added LED14: LED_0603, LED_SMD_AKL:LED_0603_1608Metric, F.Cu at (157.0, 109.9)
- added LED15: LED_0603, LED_SMD_AKL:LED_0603_1608Metric, F.Cu at (157.0, 116.1)
- added LED2: LED_0603, LED_SMD_AKL:LED_0603_1608Metric, F.Cu at (157.0, 35.5)
- added LED3: LED_0603, LED_SMD_AKL:LED_0603_1608Metric, F.Cu at (157.0, 41.7)
- added LED4: LED_0603, LED_SMD_AKL:LED_0603_1608Metric, F.Cu at (157.0, 47.9)
- added LED5: LED_0603, LED_SMD_AKL:LED_0603_1608Metric, F.Cu at (157.0, 54.1)
- added LED6: LED_0603, LED_SMD_AKL:LED_0603_1608Metric, F.Cu at (157.0, 60.3)
- added LED7: LED_0603, LED_SMD_AKL:LED_0603_1608Metric, F.Cu at (157.0, 66.5)
- added LED8: LED_0603, LED_SMD_AKL:LED_0603_1608Metric, F.Cu at (157.0, 72.7)
- added LED9: LED_0603, LED_SMD_AKL:LED_0603_1608Metric, F.Cu at (157.0, 78.9)
- added Q1: 2N7002, Package_TO_SOT_SMD_AKL:SOT-23, F.Cu at (132.2, 58.1)
- added R1: 4.7kΩ, PCM_JLCPCB:R_0603, F.Cu at (157.0, 31.5)
- added R11: 4.7kΩ, PCM_JLCPCB:R_0603, F.Cu at (157.0, 62.5)
- added R13: 4.7kΩ, PCM_JLCPCB:R_0603, F.Cu at (157.0, 68.7)
- added R18: 4.7kΩ, PCM_JLCPCB:R_0603, F.Cu at (157.0, 74.9)
- added R19: 4.7kΩ, PCM_JLCPCB:R_0603, F.Cu at (157.0, 81.1)
- added R20: 4.7kΩ, PCM_JLCPCB:R_0603, F.Cu at (157.0, 87.3)
- added R21: 4.7kΩ, PCM_JLCPCB:R_0603, F.Cu at (157.0, 93.5)
- added R22: 4.7kΩ, PCM_JLCPCB:R_0603, F.Cu at (157.0, 99.7)
- added R23: 4.7kΩ, PCM_JLCPCB:R_0603, F.Cu at (157.0, 105.9)
- added R24: 4.7kΩ, PCM_JLCPCB:R_0603, F.Cu at (157.0, 112.1)
- added R25: 4.7kΩ, PCM_JLCPCB:R_0603, F.Cu at (157.0, 118.3)
- added R26: 10k_0603, 4ms_Resistor:R_0603, F.Cu at (132.1, 55.3)
- added R27: 4.7kΩ, PCM_JLCPCB:R_0603, F.Cu at (150.9, 96.1)
- added R28: 4.7kΩ, PCM_JLCPCB:R_0603, F.Cu at (150.9, 98.3)
- added R3: 4.7kΩ, PCM_JLCPCB:R_0603, F.Cu at (157.0, 37.7)
- added R30: 10kΩ, PCM_JLCPCB:R_0603, F.Cu at (131.1, 64.5)
- added R5: 4.7kΩ, PCM_JLCPCB:R_0603, F.Cu at (157.0, 43.9)
- added R7: 4.7kΩ, PCM_JLCPCB:R_0603, F.Cu at (157.0, 50.1)
- added R9: 4.7kΩ, PCM_JLCPCB:R_0603, F.Cu at (157.0, 56.3)
- added RZ2: RP2040-Zero, Boards:RP2040-Zero_socket, F.Cu at (141.5, 104.4)
- added U3: LM1117MP-3.3, Package_TO_SOT_SMD:SOT-223-3_TabPin2, F.Cu at (125.2, 72.6)
- added U4: ENC28J60MODULE, Boards:W5500Lite-module, F.Cu at (129.7, 72.5)
- moved C10 120.4 mm to (148.7, 69.1), turned to 180 degrees
- moved C9 118.6 mm to (148.8, 45.8), turned to 180 degrees
- moved C11 113.9 mm to (145.8, 117.8), turned to -90 degrees
- moved R17 101.7 mm to (119.8, 95.2), turned to -90 degrees
- moved C12 98.0 mm to (136.8, 117.9), turned to -90 degrees
- moved D2 96.5 mm to (133.2, 110.5), turned to 90 degrees
- moved C4 79.8 mm to (147.1, 40.6), turned to 180 degrees
- moved C3 78.9 mm to (146.9, 63.9)
- moved R16 63.8 mm to (127.3, 38.3)
- moved R15 63.8 mm to (125.3, 38.3)
- moved C2 63.2 mm to (129.1, 38.3), turned to -90 degrees
- moved R14 63.0 mm to (123.6, 58.4)
- moved R8 63.0 mm to (123.6, 54.2)
- moved R2 62.6 mm to (128.7, 54.2), turned to 90 degrees
- moved R12 62.5 mm to (125.3, 58.4)
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Connections:
- J8 pad 7: unconnected-(J8-Pin_7-Pad7) -> /Relay_channel_15/NO
- J8 pad 8: unconnected-(J8-Pin_8-Pad8) -> /Relay_channel_15/COM
- J8 pad 9: unconnected-(J8-Pin_9-Pad9) -> /Relay_channel_15/NC
Routing:
- net PWR_12V: track 140.2 -> 251.0 mm, vias 0 -> 1
- net /Relay_channel_15/cntrl_A1: track 0.00 -> 79.9 mm, vias 0 -> 1
- net PWR_GND: track 121.5 -> 42.9 mm, vias 0 -> 2
- net /Relay_channel_14/cntrl_A1: track 0.00 -> 58.0 mm, vias 0 -> 1
- net /Relay_channel_13/cntrl_A1: track 0.00 -> 55.9 mm, vias 0 -> 1
- net (no net): track 41.2 -> 0.00 mm
- net /Relay_channel_12/cntrl_A1: track 11.1 -> 48.7 mm, vias 0 -> 1
- net /Relay_channel_7/NC: track 0.00 -> 37.3 mm
- net /Relay_channel_10/NC: track 0.00 -> 36.6 mm
- net /Relay_channel_11/cntrl_A1: track 10.1 -> 46.6 mm, vias 0 -> 1
- net /Relay_channel_13/NC: track 0.00 -> 35.9 mm
- net /Relay_channel_7/COM: track 0.00 -> 35.6 mm
- net /Relay_channel_10/COM: track 0.00 -> 34.3 mm
- net /Relay_channel_13/COM: track 0.00 -> 33.5 mm
- net /Relay_channel_7/NO: track 0.00 -> 32.6 mm
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Other:
- board text removed: "0"
- board text removed: "1"
- board text removed: "1+"
- board text removed: "1-"
- board text removed: "10+"
- board text removed: "2+"
- board text removed: "3+"
- board text removed: "4+"
- board text removed: "5+"
- board text removed: "6+"
- board text removed: "7+"
- board text removed: "8+"
- board text removed: "9+"
