File: 12x_relay_board/12x_relay_board.kicad_sch (KiCad schematic)
At the start: 21 parts, among them J1 Conn_01x36_MountingPin, J2 JST_03, J3 JST_03, J4 Barrel_Jack_Switch, U7 LM1117MP-3.3

Commit message: update
Parts:
- removed J1: Conn_01x36_MountingPin, Connector_PinHeader_2.54mm:PinHeader_1x36_P2.54mm_Vertical, symbol Connector_Generic_MountingPin:Conn_01x36_MountingPin
- added J1, J5, J6, J7, J8: Conn_01x09, TerminalBlock:TerminalBlock_Xinya_XY308-2.54-9P_1x09_P2.54mm_Horizontal, symbol SparkFun-Connector:Conn_01x09_P2.54mm
Connections:
- net Relay_channel_1/COM: now also J1.2 (Pin_2)
- net Relay_channel_1/NC: now also J1.3 (Pin_3)
- net Relay_channel_1/NO: now also J1.1 (Pin_1)
- net Relay_channel_10/COM: now also J7.2 (Pin_2)
- net Relay_channel_10/NC: now also J7.3 (Pin_3)
- net Relay_channel_10/NO: now also J7.1 (Pin_1)
- net Relay_channel_11/COM: now also J7.5 (Pin_5)
- net Relay_channel_11/NC: now also J7.6 (Pin_6)
- net Relay_channel_11/NO: now also J7.4 (Pin_4)
- net Relay_channel_12/COM: now also J7.8 (Pin_8)
- net Relay_channel_12/NC: now also J7.9 (Pin_9)
- net Relay_channel_12/NO: now also J7.7 (Pin_7)
- net Relay_channel_2/COM: now also J1.5 (Pin_5)
- net Relay_channel_2/NC: now also J1.6 (Pin_6)
- net Relay_channel_2/NO: now also J1.4 (Pin_4)
- net Relay_channel_3/COM: now also J1.8 (Pin_8)
- net Relay_channel_3/NC: now also J1.9 (Pin_9)
- net Relay_channel_3/NO: now also J1.7 (Pin_7)
- net Relay_channel_4/COM: now also J5.2 (Pin_2)
- net Relay_channel_4/NC: now also J5.3 (Pin_3)
- net Relay_channel_4/NO: now also J5.1 (Pin_1)
- net Relay_channel_5/COM: now also J5.5 (Pin_5)
- net Relay_channel_5/NC: now also J5.6 (Pin_6)
- net Relay_channel_5/NO: now also J5.4 (Pin_4)
- net Relay_channel_6/COM: now also J5.8 (Pin_8)
- net Relay_channel_6/NC: now also J5.9 (Pin_9)
- net Relay_channel_6/NO: now also J5.7 (Pin_7)
- net Relay_channel_7/COM: now also J6.2 (Pin_2)
- net Relay_channel_7/NC: now also J6.3 (Pin_3)
- net Relay_channel_7/NO: now also J6.1 (Pin_1)
- net Relay_channel_8/COM: now also J6.5 (Pin_5)
- net Relay_channel_8/NC: now also J6.6 (Pin_6)
- net Relay_channel_8/NO: now also J6.4 (Pin_4)
- net Relay_channel_9/COM: now also J6.8 (Pin_8)
- net Relay_channel_9/NC: now also J6.9 (Pin_9)
- net Relay_channel_9/NO: now also J6.7 (Pin_7)
- new net Relay_channel_13/COM: J8.2 (Pin_2)
- new net Relay_channel_13/NC: J8.3 (Pin_3)
- new net Relay_channel_13/NO: J8.1 (Pin_1)
- new net Relay_channel_14/COM: J8.5 (Pin_5)
- new net Relay_channel_14/NC: J8.6 (Pin_6)
- new net Relay_channel_14/NO: J8.4 (Pin_4)
Other:
- added sheet Relay_channel_13 (relay_channel.kicad_sch)
- added sheet Relay_channel_14 (relay_channel.kicad_sch)
- moved on the sheet: H1, H2, H3, H4, H5

Commit message: update
Parts:
- removed C7, C8: 100nF_0603_16V, 4ms_Capacitor:C_0603, symbol PCM_4ms_Capacitor:100nF_0603_16V
- removed D2: SS14, Diode_SMD:D_SMA, symbol Diode:SS14
- removed J4: Barrel_Jack_Switch, Connector_BarrelJack:BarrelJack_GCT_DCJ200-10-A_Horizontal, symbol Connector:Barrel_Jack_Switch
- removed R15, R16: 10k_0603, 4ms_Resistor:R_0603, symbol PCM_4ms_Resistor:10k_0603
- removed U7: LM1117MP-3.3, Package_TO_SOT_SMD:SOT-223-3_TabPin2, symbol Regulator_Linear:LM1117MP-3.3
- added D4: BAV23C, Package_TO_SOT_SMD_AKL:SOT-23, symbol Diode_AKL:BAV23C
- added Q1: 2N7002, Package_TO_SOT_SMD_AKL:SOT-23, symbol Transistor_MOSFET_AKL:2N7002
- added R26: 10k_0603, 4ms_Resistor:R_0603, symbol PCM_4ms_Resistor:10k_0603
Connections:
- net PWR_12V: now also D4.3 (K)
- net PWR_GND: now also Q1.2 (S), R26.2
- net conrol/OA0: now also Q1.1 (G), R26.1
- net Relay_channel_15/NO: now reaches J8.7 (Pin_7)
- net Relay_channel_15/COM: now reaches J8.8 (Pin_8)
- net Relay_channel_15/NC: now reaches J8.9 (Pin_9)
- new net Relay_channel_15/cntrl_A1: D4.1 (A2), D4.2 (A1), Q1.3 (D)
Other:
- added sheet ETH (Ethernet.kicad_sch)
- added sheet Power (power.kicad_sch)
- added sheet Relay_channel_15 (relay_channel.kicad_sch)
- added sheet Untitled Sheet (rp2040-zero.kicad_sch)
- sheet conrol ports: added PWR_VDD; removed none
- moved on the sheet: J1, J2, J3, J5, J6, J7, J8
