File: 12x_relay_board/control.kicad_sch (KiCad schematic)
At the start: 9 parts, among them U5 MCP23017_SO

Commit message: update
Other:
- moved on the sheet: C2

Commit message: update
Connections:
- net PWR_5V renamed PWR_VDD
Other:
- moved on the sheet: R2
