File: 12x_relay_board/relay_channel.kicad_sch (KiCad schematic)
At the start: 1 part, among them K1 FINDER-34.51

Commit message: update
Parts:
- added LED1: LED_0603, LED_SMD_AKL:LED_0603_1608Metric, symbol LED_AKL:LED_0603
- added R1: 4.7kΩ, PCM_JLCPCB:R_0603, symbol PCM_JLCPCB-Resistors:0603,4.7kΩ
Connections:
- net cntrl_A1: now also LED1.1 (K)
- net cntrl_A2: now also R1.1
- new net: LED1.2 (A), R1.2
